Commit message: Renamed op3_descrption package to orbo_description

File: orbo_ws/src/orbo_description/urdf/orbo.urdf (robot description, URDF)
Before this commit: robot robotis_op3, 13 links, 12 joints
Links:
- link body_link: geometry collision mesh filename=package://orbo_description/meshes/body.stl scale=0.001 0.001 0.001; visual mesh filename=package://orbo_description/meshes/body.stl scale=0.001 0.001 0.001
- link l_ank_pitch_link: geometry collision mesh filename=package://orbo_description/meshes/ll5.stl scale=0.001 0.001 0.001; visual mesh filename=package://orbo_description/meshes/ll5.stl scale=0.001 0.001 0.001
- link l_ank_roll_link: geometry collision mesh filename=package://orbo_description/meshes/ll6.stl scale=0.001 0.001 0.001; visual mesh filename=package://orbo_description/meshes/ll6.stl scale=0.001 0.001 0.001
- link l_hip_pitch_link: geometry collision mesh filename=package://orbo_description/meshes/ll3.stl scale=0.001 0.001 0.001; visual mesh filename=package://orbo_description/meshes/ll3.stl scale=0.001 0.001 0.001
- link l_hip_roll_link: geometry collision mesh filename=package://orbo_description/meshes/ll2.stl scale=0.001 0.001 0.001; visual mesh filename=package://orbo_description/meshes/ll2.stl scale=0.001 0.001 0.001
- link l_hip_yaw_link: geometry collision mesh filename=package://orbo_description/meshes/ll1.stl scale=0.001 0.001 0.001; visual mesh filename=package://orbo_description/meshes/ll1.stl scale=0.001 0.001 0.001
- link l_knee_link: geometry collision mesh filename=package://orbo_description/meshes/ll4.stl scale=0.001 0.001 0.001; visual mesh filename=package://orbo_description/meshes/ll4.stl scale=0.001 0.001 0.001
- link r_ank_pitch_link: geometry collision mesh filename=package://orbo_description/meshes/rl5.stl scale=0.001 0.001 0.001; visual mesh filename=package://orbo_description/meshes/rl5.stl scale=0.001 0.001 0.001
- link r_ank_roll_link: geometry collision mesh filename=package://orbo_description/meshes/rl6.stl scale=0.001 0.001 0.001; visual mesh filename=package://orbo_description/meshes/rl6.stl scale=0.001 0.001 0.001
- link r_hip_pitch_link: geometry collision mesh filename=package://orbo_description/meshes/rl3.stl scale=0.001 0.001 0.001; visual mesh filename=package://orbo_description/meshes/rl3.stl scale=0.001 0.001 0.001
- link r_hip_roll_link: geometry collision mesh filename=package://orbo_description/meshes/rl2.stl scale=0.001 0.001 0.001; visual mesh filename=package://orbo_description/meshes/rl2.stl scale=0.001 0.001 0.001
- link r_hip_yaw_link: geometry collision mesh filename=package://orbo_description/meshes/rl1.stl scale=0.001 0.001 0.001; visual mesh filename=package://orbo_description/meshes/rl1.stl scale=0.001 0.001 0.001
- link r_knee_link: geometry collision mesh filename=package://orbo_description/meshes/rl4.stl scale=0.001 0.001 0.001; visual mesh filename=package://orbo_description/meshes/rl4.stl scale=0.001 0.001 0.001

File: orbo_ws/src/orbo_description/urdf/orbo.urdf.xacro (robot description, xacro)
@@ -1,23 +1,23 @@
 <?xml version="1.0" ?>
 <robot xmlns:xacro="http://ros.org/wiki/xacro" name="robotis_op3">
-  <xacro:include filename="$(find op3_description)/urdf/orbo.visuals.xacro" />
-  <xacro:include filename="$(find op3_description)/urdf/orbo.inertia.xacro" />
-  <xacro:include filename="$(find op3_description)/urdf/robotis_op3.structure.rleg.xacro" />
-  <xacro:include filename="$(find op3_description)/urdf/robotis_op3.structure.lleg.xacro" />
+  <xacro:include filename="$(find orbo_description)/urdf/orbo.visuals.xacro" />
+  <xacro:include filename="$(find orbo_description)/urdf/orbo.inertia.xacro" />
+  <xacro:include filename="$(find orbo_description)/urdf/robotis_op3.structure.rleg.xacro" />
+  <xacro:include filename="$(find orbo_description)/urdf/robotis_op3.structure.lleg.xacro" />
   <!--
-  <xacro:include filename="$(find op3_description)/urdf/robotis_op3.structure.rarm.xacro" />
+  <xacro:include filename="$(find orbo_description)/urdf/robotis_op3.structure.rarm.xacro" />
   -->
   <!--
-  <xacro:include filename="$(find op3_description)/urdf/robotis_op3.structure.larm.xacro" />
+  <xacro:include filename="$(find orbo_description)/urdf/robotis_op3.structure.larm.xacro" />
   -->
   <!--
-  <xacro:include filename="$(find op3_description)/urdf/robotis_op3.structure.head.xacro" />
+  <xacro:include filename="$(find orbo_description)/urdf/robotis_op3.structure.head.xacro" />
   -->
   <!--
-  <xacro:include filename="$(find op3_description)/urdf/robotis_op3.gazebo.xacro" />
+  <xacro:include filename="$(find orbo_description)/urdf/robotis_op3.gazebo.xacro" />
   -->
-  <xacro:include filename="$(find op3_description)/urdf/robotis_op3.transmissions.xacro" />
+  <xacro:include filename="$(find orbo_description)/urdf/robotis_op3.transmissions.xacro" />
   <!--
-  <xacro:include filename="$(find op3_description)/urdf/gazebo_harness.xacro" />
+  <xacro:include filename="$(find orbo_description)/urdf/gazebo_harness.xacro" />
   -->
   <!-- harness link -->

File: orbo_ws/src/orbo_description/urdf/orbo.visuals.xacro (robot description, xacro)
@@ -8,5 +8,5 @@
     <origin xyz="0 0 0" rpy="0 0 0" />
     <geometry>
-      <mesh filename="package://op3_description/meshes/body.stl"  scale="0.001 0.001 0.001"/>
+      <mesh filename="package://orbo_description/meshes/body.stl"  scale="0.001 0.001 0.001"/>
     </geometry>
     <material name="Grey">
@@ -18,5 +18,5 @@
     <origin xyz="0 0 0" rpy="0 0 0" />
     <geometry>
-      <mesh filename="package://op3_description/meshes/rl1.stl"  scale="0.001 0.001 0.001"/>
+      <mesh filename="package://orbo_description/meshes/rl1.stl"  scale="0.001 0.001 0.001"/>
     </geometry>
     <material name="Grey">
@@ -28,5 +28,5 @@
     <origin xyz="0 0 0" rpy="0 0 0" />
     <geometry>
-      <mesh filename="package://op3_description/meshes/rl2.stl"  scale="0.001 0.001 0.001"/>
+      <mesh filename="package://orbo_description/meshes/rl2.stl"  scale="0.001 0.001 0.001"/>
     </geometry>
     <material name="Grey">
@@ -38,5 +38,5 @@
     <origin xyz="0 0 0" rpy="0 0 0" />
     <geometry>
-      <mesh filename="package://op3_description/meshes/rl3.stl"  scale="0.001 0.001 0.001"/>
+      <mesh filename="package://orbo_description/meshes/rl3.stl"  scale="0.001 0.001 0.001"/>
     </geometry>
     <material name="Grey">
@@ -48,5 +48,5 @@
     <origin xyz="0 0 0" rpy="0 0 0" />
     <geometry>
-      <mesh filename="package://op3_description/meshes/rl4.stl"  scale="0.001 0.001 0.001"/>
+      <mesh filename="package://orbo_description/meshes/rl4.stl"  scale="0.001 0.001 0.001"/>
     </geometry>
     <material name="Grey">
@@ -58,5 +58,5 @@
     <origin xyz="0 0 0" rpy="0 0 0" />
     <geometry>
-      <mesh filename="package://op3_description/meshes/rl5.stl"  scale="0.001 0.001 0.001"/>
+      <mesh filename="package://orbo_description/meshes/rl5.stl"  scale="0.001 0.001 0.001"/>
     </geometry>
     <material name="Grey">
@@ -68,5 +68,5 @@
     <origin xyz="0 0 0" rpy="0 0 0" />
     <geometry>
-      <mesh filename="package://op3_description/meshes/rl6.stl"  scale="0.001 0.001 0.001"/>
+      <mesh filename="package://orbo_description/meshes/rl6.stl"  scale="0.001 0.001 0.001"/>
     </geometry>
     <material name="Grey">
@@ -78,5 +78,5 @@
     <origin xyz="0 0 0" rpy="0 0 0" />
     <geometry>
-      <mesh filename="package://op3_description/meshes/ll1.stl"  scale="0.001 0.001 0.001"/>
+      <mesh filename="package://orbo_description/meshes/ll1.stl"  scale="0.001 0.001 0.001"/>
     </geometry>
     <material name="Grey">
@@ -88,5 +88,5 @@
     <origin xyz="0 0 0" rpy="0 0 0" />
     <geometry>
-      <mesh filename="package://op3_description/meshes/ll2.stl"  scale="0.001 0.001 0.001"/>
+      <mesh filename="package://orbo_description/meshes/ll2.stl"  scale="0.001 0.001 0.001"/>
     </geometry>
     <material name="Grey">
@@ -98,5 +98,5 @@
     <origin xyz="0 0 0" rpy="0 0 0" />
     <geometry>
-      <mesh filename="package://op3_description/meshes/ll3.stl"  scale="0.001 0.001 0.001"/>
+      <mesh filename="package://orbo_description/meshes/ll3.stl"  scale="0.001 0.001 0.001"/>
     </geometry>
     <material name="Grey">
@@ -108,5 +108,5 @@
     <origin xyz="0 0 0" rpy="0 0 0" />
     <geometry>
-      <mesh filename="package://op3_description/meshes/ll4.stl"  scale="0.001 0.001 0.001"/>
+      <mesh filename="package://orbo_description/meshes/ll4.stl"  scale="0.001 0.001 0.001"/>
     </geometry>
     <material name="Grey">
@@ -118,5 +118,5 @@
     <origin xyz="0 0 0" rpy="0 0 0" />
     <geometry>
-      <mesh filename="package://op3_description/meshes/ll5.stl"  scale="0.001 0.001 0.001"/>
+      <mesh filename="package://orbo_description/meshes/ll5.stl"  scale="0.001 0.001 0.001"/>
     </geometry>
     <material name="Grey">
@@ -128,89 +128,97 @@
     <origin xyz="0 0 0" rpy="0 0 0" />
     <geometry>
-      <mesh filename="package://op3_description/meshes/ll6.stl"  scale="0.001 0.001 0.001"/>
-    </geometry>
-    <material name="Grey">
-      <color rgba="0.60 0.60 0.60 1.0"/>
-    </material>
-  </xacro:macro>
-  <!-- right shoulder pitch joint -->
+      <mesh filename="package://orbo_description/meshes/ll6.stl"  scale="0.001 0.001 0.001"/>
+    </geometry>
+    <material name="Grey">
+      <color rgba="0.60 0.60 0.60 1.0"/>
+    </material>
+  </xacro:macro>
+  <!-- right shoulder pitch joint
   <xacro:macro name="insert_mesh_r_sho_pitch_link">
     <origin xyz="0 0 0" rpy="0 0 0" />
     <geometry>
-      <mesh filename="package://op3_description/meshes/ra1.stl"  scale="0.001 0.001 0.001"/>
-    </geometry>
-    <material name="Grey">
-      <color rgba="0.60 0.60 0.60 1.0"/>
-    </material>
-  </xacro:macro>
-  <!-- right shoulder pitch joint -->
+      <mesh filename="package://orbo_description/meshes/ra1.stl"  scale="0.001 0.001 0.001"/>
+    </geometry>
+    <material name="Grey">
+      <color rgba="0.60 0.60 0.60 1.0"/>
+    </material>
+  </xacro:macro>
+  -->
+  <!-- right shoulder pitch joint
   <xacro:macro name="insert_mesh_r_sho_roll_link">
     <origin xyz="0 0 0" rpy="0 0 0" />
     <geometry>
-      <mesh filename="package://op3_description/meshes/ra2.stl"  scale="0.001 0.001 0.001"/>
-    </geometry>
-    <material name="Grey">
-      <color rgba="0.60 0.60 0.60 1.0"/>
-    </material>
-  </xacro:macro>
-  <!-- right elbow joint -->
+      <mesh filename="package://orbo_description/meshes/ra2.stl"  scale="0.001 0.001 0.001"/>
+    </geometry>
+    <material name="Grey">
+      <color rgba="0.60 0.60 0.60 1.0"/>
+    </material>
+  </xacro:macro>
+  -->
+  <!-- right elbow joint
   <xacro:macro name="insert_mesh_r_el_link">
     <origin xyz="0 0 0" rpy="0 0 0" />
     <geometry>
-      <mesh filename="package://op3_description/meshes/ra3.stl"  scale="0.001 0.001 0.001"/>
-    </geometry>
-    <material name="Grey">
-      <color rgba="0.60 0.60 0.60 1.0"/>
-    </material>
-  </xacro:macro>
-  <!-- left shoulder pitch joint -->
+      <mesh filename="package://orbo_description/meshes/ra3.stl"  scale="0.001 0.001 0.001"/>
+    </geometry>
+    <material name="Grey">
+      <color rgba="0.60 0.60 0.60 1.0"/>
+    </material>
+  </xacro:macro>
+  -->
+  <!-- left shoulder pitch joint
   <xacro:macro name="insert_mesh_l_sho_pitch_link">
     <origin xyz="0 0 0" rpy="0 0 0" />
     <geometry>
-      <mesh filename="package://op3_description/meshes/la1.stl"  scale="0.001 0.001 0.001"/>
-    </geometry>
-    <material name="Grey">
-      <color rgba="0.60 0.60 0.60 1.0"/>
-    </material>
-  </xacro:macro>
-  <!-- left shoulder pitch joint -->
+      <mesh filename="package://orbo_description/meshes/la1.stl"  scale="0.001 0.001 0.001"/>
+    </geometry>
+    <material name="Grey">
+      <color rgba="0.60 0.60 0.60 1.0"/>
+    </material>
+  </xacro:macro>
+  -->
+  <!-- left shoulder pitch joint
   <xacro:macro name="insert_mesh_l_sho_roll_link">
     <origin xyz="0 0 0" rpy="0 0 0" />
     <geometry>
-      <mesh filename="package://op3_description/meshes/la2.stl"  scale="0.001 0.001 0.001"/>
-    </geometry>
-    <material name="Grey">
-      <color rgba="0.60 0.60 0.60 1.0"/>
-    </material>
-  </xacro:macro>
-  <!-- left elbow joint -->
+      <mesh filename="package://orbo_description/meshes/la2.stl"  scale="0.001 0.001 0.001"/>
+    </geometry>
+    <material name="Grey">
+      <color rgba="0.60 0.60 0.60 1.0"/>
+    </material>
+  </xacro:macro>
+  -->
+  <!-- left elbow joint
   <xacro:macro name="insert_mesh_l_el_link">
     <origin xyz="0 0 0" rpy="0 0 0" />
     <geometry>
-      <mesh filename="package://op3_description/meshes/la3.stl"  scale="0.001 0.001 0.001"/>
-    </geometry>
-    <material name="Grey">
-      <color rgba="0.60 0.60 0.60 1.0"/>
-    </material>
-  </xacro:macro>
-  <!-- head yaw joint -->
+      <mesh filename="package://orbo_description/meshes/la3.stl"  scale="0.001 0.001 0.001"/>
+    </geometry>
+    <material name="Grey">
+      <color rgba="0.60 0.60 0.60 1.0"/>
+    </material>
+  </xacro:macro>
+  -->
+  <!-- head yaw joint
   <xacro:macro name="insert_mesh_head_pan_link">
     <origin xyz="0 0 0" rpy="0 0 0" />
     <geometry>
-      <mesh filename="package://op3_description/meshes/h1.stl"  scale="0.001 0.001 0.001"/>
-    </geometry>
-    <material name="Grey">
-      <color rgba="0.60 0.60 0.60 1.0"/>
-    </material>
-  </xacro:macro>
-  <!-- head yaw joint -->
+      <mesh filename="package://orbo_description/meshes/h1.stl"  scale="0.001 0.001 0.001"/>
+    </geometry>
+    <material name="Grey">
+      <color rgba="0.60 0.60 0.60 1.0"/>
+    </material>
+  </xacro:macro>
+  -->
+  <!-- head yaw joint
   <xacro:macro name="insert_mesh_head_tilt_link">
     <origin xyz="0 0 0" rpy="0 0 0" />
     <geometry>
-      <mesh filename="package://op3_description/meshes/h2.stl"  scale="0.001 0.001 0.001"/>
-    </geometry>
-    <material name="Grey">
-      <color rgba="0.60 0.60 0.60 1.0"/>
-    </material>
-  </xacro:macro>
+      <mesh filename="package://orbo_description/meshes/h2.stl"  scale="0.001 0.001 0.001"/>
+    </geometry>
+    <material name="Grey">
+      <color rgba="0.60 0.60 0.60 1.0"/>
+    </material>
+  </xacro:macro>
+  -->
 </robot>

File: orbo_ws/src/orbo_description/urdf/robotis_op3.urdf.xacro (robot description, xacro)
@@ -1,15 +1,15 @@
 <?xml version="1.0" ?>
 <robot xmlns:xacro="http://ros.org/wiki/xacro" name="robotis_op3">
-  <xacro:include filename="$(find op3_description)/urdf/robotis_op3.visuals.xacro" />
-  <xacro:include filename="$(find op3_description)/urdf/robotis_op3.inertia.xacro" />
-  <xacro:include filename="$(find op3_description)/urdf/robotis_op3.structure.rleg.xacro" />
-  <xacro:include filename="$(find op3_description)/urdf/robotis_op3.structure.lleg.xacro" />
-  <xacro:include filename="$(find op3_description)/urdf/robotis_op3.structure.rarm.xacro" />
-  <xacro:include filename="$(find op3_description)/urdf/robotis_op3.structure.larm.xacro" />
-  <xacro:include filename="$(find op3_description)/urdf/robotis_op3.structure.head.xacro" />
-  <xacro:include filename="$(find op3_description)/urdf/robotis_op3.gazebo.xacro" />
-  <xacro:include filename="$(find op3_description)/urdf/robotis_op3.transmissions.xacro" />
+  <xacro:include filename="$(find orbo_description)/urdf/robotis_op3.visuals.xacro" />
+  <xacro:include filename="$(find orbo_description)/urdf/robotis_op3.inertia.xacro" />
+  <xacro:include filename="$(find orbo_description)/urdf/robotis_op3.structure.rleg.xacro" />
+  <xacro:include filename="$(find orbo_description)/urdf/robotis_op3.structure.lleg.xacro" />
+  <xacro:include filename="$(find orbo_description)/urdf/robotis_op3.structure.rarm.xacro" />
+  <xacro:include filename="$(find orbo_description)/urdf/robotis_op3.structure.larm.xacro" />
+  <xacro:include filename="$(find orbo_description)/urdf/robotis_op3.structure.head.xacro" />
+  <xacro:include filename="$(find orbo_description)/urdf/robotis_op3.gazebo.xacro" />
+  <xacro:include filename="$(find orbo_description)/urdf/robotis_op3.transmissions.xacro" />
   <!--
-  <xacro:include filename="$(find op3_description)/urdf/gazebo_harness.xacro" />
+  <xacro:include filename="$(find orbo_description)/urdf/gazebo_harness.xacro" />
   -->
   <!-- harness link -->
