Commit message: Renamed op3_descrption package to orbo_description

File: orbo_ws/src/orbo_description/urdf/robotis_op3.visuals.xacro (robot description, xacro)
@@ -8,5 +8,5 @@
     <origin xyz="0 0 0" rpy="0 0 0" />
     <geometry>
-      <mesh filename="package://op3_description/meshes/body.stl"  scale="0.001 0.001 0.001"/>
+      <mesh filename="package://orbo_description/meshes/body.stl"  scale="0.001 0.001 0.001"/>
     </geometry>
     <material name="Grey">
@@ -18,5 +18,5 @@
     <origin xyz="0 0 0" rpy="0 0 0" />
     <geometry>
-      <mesh filename="package://op3_description/meshes/rl1.stl"  scale="0.001 0.001 0.001"/>
+      <mesh filename="package://orbo_description/meshes/rl1.stl"  scale="0.001 0.001 0.001"/>
     </geometry>
     <material name="Grey">
@@ -28,5 +28,5 @@
     <origin xyz="0 0 0" rpy="0 0 0" />
     <geometry>
-      <mesh filename="package://op3_description/meshes/rl2.stl"  scale="0.001 0.001 0.001"/>
+      <mesh filename="package://orbo_description/meshes/rl2.stl"  scale="0.001 0.001 0.001"/>
     </geometry>
     <material name="Grey">
@@ -38,5 +38,5 @@
     <origin xyz="0 0 0" rpy="0 0 0" />
     <geometry>
-      <mesh filename="package://op3_description/meshes/rl3.stl"  scale="0.001 0.001 0.001"/>
+      <mesh filename="package://orbo_description/meshes/rl3.stl"  scale="0.001 0.001 0.001"/>
     </geometry>
     <material name="Grey">
@@ -48,5 +48,5 @@
     <origin xyz="0 0 0" rpy="0 0 0" />
     <geometry>
-      <mesh filename="package://op3_description/meshes/rl4.stl"  scale="0.001 0.001 0.001"/>
+      <mesh filename="package://orbo_description/meshes/rl4.stl"  scale="0.001 0.001 0.001"/>
     </geometry>
     <material name="Grey">
@@ -58,5 +58,5 @@
     <origin xyz="0 0 0" rpy="0 0 0" />
     <geometry>
-      <mesh filename="package://op3_description/meshes/rl5.stl"  scale="0.001 0.001 0.001"/>
+      <mesh filename="package://orbo_description/meshes/rl5.stl"  scale="0.001 0.001 0.001"/>
     </geometry>
     <material name="Grey">
@@ -68,5 +68,5 @@
     <origin xyz="0 0 0" rpy="0 0 0" />
     <geometry>
-      <mesh filename="package://op3_description/meshes/rl6.stl"  scale="0.001 0.001 0.001"/>
+      <mesh filename="package://orbo_description/meshes/rl6.stl"  scale="0.001 0.001 0.001"/>
     </geometry>
     <material name="Grey">
@@ -78,5 +78,5 @@
     <origin xyz="0 0 0" rpy="0 0 0" />
     <geometry>
-      <mesh filename="package://op3_description/meshes/ll1.stl"  scale="0.001 0.001 0.001"/>
+      <mesh filename="package://orbo_description/meshes/ll1.stl"  scale="0.001 0.001 0.001"/>
     </geometry>
     <material name="Grey">
@@ -88,5 +88,5 @@
     <origin xyz="0 0 0" rpy="0 0 0" />
     <geometry>
-      <mesh filename="package://op3_description/meshes/ll2.stl"  scale="0.001 0.001 0.001"/>
+      <mesh filename="package://orbo_description/meshes/ll2.stl"  scale="0.001 0.001 0.001"/>
     </geometry>
     <material name="Grey">
@@ -98,5 +98,5 @@
     <origin xyz="0 0 0" rpy="0 0 0" />
     <geometry>
-      <mesh filename="package://op3_description/meshes/ll3.stl"  scale="0.001 0.001 0.001"/>
+      <mesh filename="package://orbo_description/meshes/ll3.stl"  scale="0.001 0.001 0.001"/>
     </geometry>
     <material name="Grey">
@@ -108,5 +108,5 @@
     <origin xyz="0 0 0" rpy="0 0 0" />
     <geometry>
-      <mesh filename="package://op3_description/meshes/ll4.stl"  scale="0.001 0.001 0.001"/>
+      <mesh filename="package://orbo_description/meshes/ll4.stl"  scale="0.001 0.001 0.001"/>
     </geometry>
     <material name="Grey">
@@ -118,5 +118,5 @@
     <origin xyz="0 0 0" rpy="0 0 0" />
     <geometry>
-      <mesh filename="package://op3_description/meshes/ll5.stl"  scale="0.001 0.001 0.001"/>
+      <mesh filename="package://orbo_description/meshes/ll5.stl"  scale="0.001 0.001 0.001"/>
     </geometry>
     <material name="Grey">
@@ -128,97 +128,89 @@
     <origin xyz="0 0 0" rpy="0 0 0" />
     <geometry>
-      <mesh filename="package://op3_description/meshes/ll6.stl"  scale="0.001 0.001 0.001"/>
-    </geometry>
-    <material name="Grey">
-      <color rgba="0.60 0.60 0.60 1.0"/>
-    </material>
-  </xacro:macro>
-  <!-- right shoulder pitch joint
+      <mesh filename="package://orbo_description/meshes/ll6.stl"  scale="0.001 0.001 0.001"/>
+    </geometry>
+    <material name="Grey">
+      <color rgba="0.60 0.60 0.60 1.0"/>
+    </material>
+  </xacro:macro>
+  <!-- right shoulder pitch joint -->
   <xacro:macro name="insert_mesh_r_sho_pitch_link">
     <origin xyz="0 0 0" rpy="0 0 0" />
     <geometry>
-      <mesh filename="package://op3_description/meshes/ra1.stl"  scale="0.001 0.001 0.001"/>
-    </geometry>
-    <material name="Grey">
-      <color rgba="0.60 0.60 0.60 1.0"/>
-    </material>
-  </xacro:macro>
-  -->
-  <!-- right shoulder pitch joint
+      <mesh filename="package://orbo_description/meshes/ra1.stl"  scale="0.001 0.001 0.001"/>
+    </geometry>
+    <material name="Grey">
+      <color rgba="0.60 0.60 0.60 1.0"/>
+    </material>
+  </xacro:macro>
+  <!-- right shoulder pitch joint -->
   <xacro:macro name="insert_mesh_r_sho_roll_link">
     <origin xyz="0 0 0" rpy="0 0 0" />
     <geometry>
-      <mesh filename="package://op3_description/meshes/ra2.stl"  scale="0.001 0.001 0.001"/>
-    </geometry>
-    <material name="Grey">
-      <color rgba="0.60 0.60 0.60 1.0"/>
-    </material>
-  </xacro:macro>
-  -->
-  <!-- right elbow joint
+      <mesh filename="package://orbo_description/meshes/ra2.stl"  scale="0.001 0.001 0.001"/>
+    </geometry>
+    <material name="Grey">
+      <color rgba="0.60 0.60 0.60 1.0"/>
+    </material>
+  </xacro:macro>
+  <!-- right elbow joint -->
   <xacro:macro name="insert_mesh_r_el_link">
     <origin xyz="0 0 0" rpy="0 0 0" />
     <geometry>
-      <mesh filename="package://op3_description/meshes/ra3.stl"  scale="0.001 0.001 0.001"/>
-    </geometry>
-    <material name="Grey">
-      <color rgba="0.60 0.60 0.60 1.0"/>
-    </material>
-  </xacro:macro>
-  -->
-  <!-- left shoulder pitch joint
+      <mesh filename="package://orbo_description/meshes/ra3.stl"  scale="0.001 0.001 0.001"/>
+    </geometry>
+    <material name="Grey">
+      <color rgba="0.60 0.60 0.60 1.0"/>
+    </material>
+  </xacro:macro>
+  <!-- left shoulder pitch joint -->
   <xacro:macro name="insert_mesh_l_sho_pitch_link">
     <origin xyz="0 0 0" rpy="0 0 0" />
     <geometry>
-      <mesh filename="package://op3_description/meshes/la1.stl"  scale="0.001 0.001 0.001"/>
-    </geometry>
-    <material name="Grey">
-      <color rgba="0.60 0.60 0.60 1.0"/>
-    </material>
-  </xacro:macro>
-  -->
-  <!-- left shoulder pitch joint
+      <mesh filename="package://orbo_description/meshes/la1.stl"  scale="0.001 0.001 0.001"/>
+    </geometry>
+    <material name="Grey">
+      <color rgba="0.60 0.60 0.60 1.0"/>
+    </material>
+  </xacro:macro>
+  <!-- left shoulder pitch joint -->
   <xacro:macro name="insert_mesh_l_sho_roll_link">
     <origin xyz="0 0 0" rpy="0 0 0" />
     <geometry>
-      <mesh filename="package://op3_description/meshes/la2.stl"  scale="0.001 0.001 0.001"/>
-    </geometry>
-    <material name="Grey">
-      <color rgba="0.60 0.60 0.60 1.0"/>
-    </material>
-  </xacro:macro>
-  -->
-  <!-- left elbow joint
+      <mesh filename="package://orbo_description/meshes/la2.stl"  scale="0.001 0.001 0.001"/>
+    </geometry>
+    <material name="Grey">
+      <color rgba="0.60 0.60 0.60 1.0"/>
+    </material>
+  </xacro:macro>
+  <!-- left elbow joint -->
   <xacro:macro name="insert_mesh_l_el_link">
     <origin xyz="0 0 0" rpy="0 0 0" />
     <geometry>
-      <mesh filename="package://op3_description/meshes/la3.stl"  scale="0.001 0.001 0.001"/>
-    </geometry>
-    <material name="Grey">
-      <color rgba="0.60 0.60 0.60 1.0"/>
-    </material>
-  </xacro:macro>
-  -->
-  <!-- head yaw joint
+      <mesh filename="package://orbo_description/meshes/la3.stl"  scale="0.001 0.001 0.001"/>
+    </geometry>
+    <material name="Grey">
+      <color rgba="0.60 0.60 0.60 1.0"/>
+    </material>
+  </xacro:macro>
+  <!-- head yaw joint -->
   <xacro:macro name="insert_mesh_head_pan_link">
     <origin xyz="0 0 0" rpy="0 0 0" />
     <geometry>
-      <mesh filename="package://op3_description/meshes/h1.stl"  scale="0.001 0.001 0.001"/>
-    </geometry>
-    <material name="Grey">
-      <color rgba="0.60 0.60 0.60 1.0"/>
-    </material>
-  </xacro:macro>
-  -->
-  <!-- head yaw joint
+      <mesh filename="package://orbo_description/meshes/h1.stl"  scale="0.001 0.001 0.001"/>
+    </geometry>
+    <material name="Grey">
+      <color rgba="0.60 0.60 0.60 1.0"/>
+    </material>
+  </xacro:macro>
+  <!-- head yaw joint -->
   <xacro:macro name="insert_mesh_head_tilt_link">
     <origin xyz="0 0 0" rpy="0 0 0" />
     <geometry>
-      <mesh filename="package://op3_description/meshes/h2.stl"  scale="0.001 0.001 0.001"/>
-    </geometry>
-    <material name="Grey">
-      <color rgba="0.60 0.60 0.60 1.0"/>
-    </material>
-  </xacro:macro>
-  -->
+      <mesh filename="package://orbo_description/meshes/h2.stl"  scale="0.001 0.001 0.001"/>
+    </geometry>
+    <material name="Grey">
+      <color rgba="0.60 0.60 0.60 1.0"/>
+    </material>
+  </xacro:macro>
 </robot>
